Commit message: added xbox control teleop

File: red_robot_base/urdf/red_robot.xacro (robot description, xacro)
@@ -7,40 +7,30 @@
   <!-- Base Link -->
   <link name="base_link">
-    <collision>
-      <origin xyz="-0.15 0 0.1" rpy="0 0 0"/>
+    <visual>
+      <origin xyz="-0.02 0 0.05" rpy="0 0 0"/>
       <geometry>
-	    <box size=".485 .43 .15"/>
+	    <box size=".16 .11 .01"/>
       </geometry>
-    </collision>
-    <visual>
-      <origin xyz="-0.15 0 0.1" rpy="0 0 0"/>
+      <material name="red"/>
+    </visual>
+  </link>
+  <link name="caster">
+    <visual name="visual">
+      <origin xyz="-0.09 0.0 0.01" rpy="0 0 0"/>
       <geometry>
-	    <box size=".485 .43 .15"/>
+        <sphere  radius="0.01"/>
       </geometry>
-      <material name="orange"/>
+      <material name="grey"/>
     </visual>
-    <collision name="collision">
-      <origin xyz="-0.325 0.0 0.05" rpy="0 1.5707 1.5707"/>
-      <geometry>
-        <cylinder  length="0.03" radius="0.04625"/>
-      </geometry>
-    </collision>
-    <visual name="visual">
-      <origin xyz="-0.325 0.0 0.05" rpy="0 1.5707 1.5707"/>
-      <geometry>
-        <cylinder  length="0.03" radius="0.04625"/>
-      </geometry>
-    </visual>
-    <inertial>
-       <mass value="20" />
-       <origin xyz="-0.08 0 0" rpy="0 0 0"/>
-       <inertia ixx="1" ixy="0" ixz="0" iyy="1" iyz="0" izz="1" />
-    </inertial>
   </link>
+  <joint type="fixed" name="caster_joint">
+    <child link="caster">caster</child>
+    <parent link="base_link">base_link</parent>
+  </joint>
   <link name="left_wheel">
     <collision name="collision">
       <origin xyz="0 0.0 0" rpy="0 1.5707 1.5707"/>
       <geometry>
-         <cylinder  length="0.03" radius="0.0725"/>
+         <cylinder  length="0.03" radius="0.03"/>
       </geometry>
     </collision>
@@ -48,15 +38,11 @@
       <origin xyz="0 0.0 0" rpy="0 1.5707 1.5707"/>
       <geometry>
-        <cylinder  length="0.03" radius="0.0725"/>
+        <cylinder  length="0.03" radius="0.03"/>
       </geometry>
+      <material name="black"/>
     </visual>
-    <inertial>
-      <mass value="1" />
-      <origin xyz="0 0.0 0"/>
-      <inertia ixx="0.1" ixy="0" ixz="0" iyy="0.1" iyz="0" izz="0.1" />
-    </inertial>
   </link>
   <joint type="revolute" name="left_wheel_joint">
-    <origin xyz="0 0.15 0.075" rpy="0 0 0"/>
+    <origin xyz="0 0.05 0.03" rpy="0 0 0"/>
     <child link="left_wheel">left_wheel</child>
     <parent link="base_link">base_link</parent>
@@ -68,5 +54,5 @@
       <origin xyz="0 0.0 0" rpy="0 1.5707 1.5707"/>
       <geometry>
-         <cylinder  length="0.03" radius="0.0725"/>
+         <cylinder  length="0.03" radius="0.03"/>
       </geometry>
     </collision>
@@ -74,15 +60,11 @@
       <origin xyz="0 0.0 0" rpy="0 1.5707 1.5707"/>
       <geometry>
-        <cylinder  length="0.03" radius="0.0725"/>
+        <cylinder  length="0.03" radius="0.03"/>
       </geometry>
+      <material name="black"/>
     </visual>
-    <inertial>
-      <mass value="1" />
-      <origin xyz="0 0.0 0"/>
-      <inertia ixx="0.1" ixy="0" ixz="0" iyy="0.1" iyz="0" izz="0.1" />
-    </inertial>
   </link>
   <joint type="revolute" name="right_wheel_joint">
-    <origin xyz="0 -0.15 0.075" rpy="0 0 0"/>
+    <origin xyz="0 -0.05 0.03" rpy="0 0 0"/>
     <child link="right_wheel">right_wheel</child>
     <parent link="base_link">base_link</parent>

Commit message: red robot driver improvements

File: red_robot_base/urdf/red_robot.xacro (robot description, xacro)
@@ -7,5 +7,5 @@
   <!-- Base Link -->
   <link name="base_link">
-    <visual>
+    <visual name="top_plate">
       <origin xyz="-0.02 0 0.05" rpy="0 0 0"/>
       <geometry>
@@ -14,7 +14,5 @@
       <material name="red"/>
     </visual>
-  </link>
-  <link name="caster">
-    <visual name="visual">
+    <visual name="caster">
       <origin xyz="-0.09 0.0 0.01" rpy="0 0 0"/>
       <geometry>
@@ -24,8 +22,4 @@
     </visual>
   </link>
-  <joint type="fixed" name="caster_joint">
-    <child link="caster">caster</child>
-    <parent link="base_link">base_link</parent>
-  </joint>
   <link name="left_wheel">
     <collision name="collision">
@@ -72,3 +66,17 @@
     <limit effort="100" velocity="100.0"  lower="-5000" upper="5000" />
   </joint>
+  <link name="laser">
+    <visual>
+      <origin xyz="0 0.0 0" rpy="0 0 0"/>
+      <geometry>
+        <cylinder length="0.05" radius="0.03"/>
+      </geometry>
+      <material name="black"/>
+    </visual>
+  </link>
+  <joint type="fixed" name="laser_to_base_joint">
+    <origin rpy="0 0 0" xyz="0 0 0.05"/>
+    <child link="laser"/>
+    <parent link="base_link"/>
+  </joint>
 </robot>

Commit message: added imu to red robot

File: red_robot_base/urdf/red_robot.xacro (robot description, xacro)
@@ -76,7 +76,21 @@
   </link>
   <joint type="fixed" name="laser_to_base_joint">
-    <origin rpy="0 0 0" xyz="0 0 0.05"/>
+    <origin rpy="0 0 0" xyz="-0.05 0 0.05"/>
     <child link="laser"/>
     <parent link="base_link"/>
   </joint>
+  <link name="imu">
+    <visual>
+      <origin xyz="0 0.0 0" rpy="0 0 0"/>
+      <geometry>
+        <cylinder length="0.01" radius="0.01"/>
+      </geometry>
+      <material name="black"/>
+    </visual>
+  </link>
+  <joint type="fixed" name="imu_to_base_joint">
+    <origin rpy="0 0 -1.5708" xyz="0 0 0.06"/>
+    <child link="imu"/>
+    <parent link="base_link"/>
+  </joint>
 </robot>
