Commit message: Added laser to box_bot urdf

File: office_bot/urdf/box_bot.xacro (robot description, xacro)
@@ -8,5 +8,5 @@
   <link name="base_link">
     <visual name="box">
-      <origin rpy="0  0  0" xyz="-0.08181  0       0.1834"/>
+      <origin rpy="0 0 0" xyz="-0.18 0 0.185"/>
       <geometry>
         <box size="0.4 0.24 0.23"/>
@@ -15,5 +15,5 @@
     </visual>
     <visual name="left_caster">
-      <origin rpy="1.5708  0      0" xyz="-0.24564  0.11109 0.035"/>
+      <origin rpy="1.5708 0 0" xyz="-0.34500  0.11109 0.035"/>
       <geometry>
         <cylinder length="0.01" radius="0.035"/>
@@ -21,5 +21,5 @@
     </visual>
     <visual name="right_caster">
-      <origin rpy="1.5708  0      0" xyz="-0.24564 -0.11109 0.035"/>
+      <origin rpy="1.5708 0 0" xyz="-0.34500 -0.11109 0.035"/>
       <geometry>
         <cylinder length="0.01" radius="0.035"/>
@@ -27,5 +27,5 @@
     </visual>
     <visual name="neck">
-      <origin rpy="0  0  0" xyz="0.16818  0       0.0734"/>
+      <origin rpy="0 0 0" xyz="0.06 0 0.0725"/>
       <geometry>
         <box size="0.12 0.025 0.005"/>
@@ -33,5 +33,5 @@
     </visual>
     <visual name="head">
-      <origin rpy="0  0  0" xyz="0.2079   0       0.07958"/>
+      <origin rpy="0 0 0" xyz="0.12 0 0.085"/>
       <geometry>
         <box size="0.07 0.07 0.03"/>
@@ -69,6 +69,15 @@
     </visual>
   </link>
+  <link name="laser">
+    <visual>
+      <origin xyz="0 0.0 0" rpy="0 0 0"/>
+      <geometry>
+        <cylinder length="0.05" radius="0.03"/>
+      </geometry>
+      <material name="black"/>
+    </visual>
+  </link>
   <joint type="revolute" name="motor_1_joint">
-    <origin rpy="0 0 0" xyz="0.09818 -0.13 0.045"/>
+    <origin rpy="0 0 0" xyz="0.0 -0.13 0.045"/>
     <child link="right_wheel_link">right_wheel</child>
     <parent link="base_link">base_link</parent>
@@ -77,5 +86,5 @@
   </joint>
   <joint type="revolute" name="motor_2_joint">
-    <origin rpy="0 0 0" xyz="0.09818 0.13 0.045"/>
+    <origin rpy="0 0 0" xyz="0.0 0.13 0.045"/>
     <child link="left_wheel_link">left_wheel</child>
     <parent link="base_link">base_link</parent>
@@ -83,3 +92,8 @@
     <limit effort="100" velocity="100.0"  lower="-5000" upper="5000" />
   </joint>
+  <joint type="fixed" name="laser_to_base_joint">
+    <origin rpy="0 0 0" xyz="0.12 0 0.095"/>
+    <child link="laser"/>
+    <parent link="base_link"/>
+  </joint>
 </robot>

Commit message: update nav stack to not use a map

File: office_bot/urdf/box_bot.xacro (robot description, xacro)
@@ -102,5 +102,5 @@
   </joint>
   <joint type="fixed" name="base_to_laser_joint">
-    <origin rpy="0 1.571 1.571" xyz="0.12 0 0.095"/>
+    <origin rpy="0 0 0" xyz="0.12 0 0.095"/>
     <child link="laser"/>
     <parent link="base_link"/>

Commit message: Added tango urdf links

File: office_bot/urdf/box_bot.xacro (robot description, xacro)
@@ -78,4 +78,13 @@
     </visual>
   </link>
+  <link name="tango">
+    <visual>
+      <origin xyz="0 0.0 0" rpy="0 0 0"/>
+      <geometry>
+         <box size="0.2 0.12 0.01"/>
+      </geometry>
+      <material name="black"/>
+    </visual>
+  </link>
   <joint type="revolute" name="motor_1_joint">
     <origin rpy="0 0 0" xyz="0.0 -0.13 0.045"/>
@@ -92,8 +101,13 @@
     <limit effort="100" velocity="100.0"  lower="-5000" upper="5000" />
   </joint>
-  <joint type="fixed" name="laser_to_base_joint">
-    <origin rpy="0 0 0" xyz="0.12 0 0.095"/>
+  <joint type="fixed" name="base_to_laser_joint">
+    <origin rpy="0 1.571 1.571" xyz="0.12 0 0.095"/>
     <child link="laser"/>
     <parent link="base_link"/>
   </joint>
+  <joint type="fixed" name="tango_to_base_joint">
+    <origin rpy="0 1.571 1.571" xyz="0 -0.195 0.12"/>
+    <child link="base_link"/>
+    <parent link="tango"/>
+  </joint>
 </robot>

Commit message: Corrected tf heights in tango_nav_adaptor

File: office_bot/urdf/box_bot.xacro (robot description, xacro)
@@ -69,5 +69,5 @@
     </visual>
   </link>
-  <link name="laser">
+  <link name="laser_link">
     <visual>
       <origin xyz="0 0.0 0" rpy="0 0 0"/>
@@ -101,7 +101,7 @@
     <limit effort="100" velocity="100.0"  lower="-5000" upper="5000" />
   </joint>
-  <joint type="fixed" name="base_to_laser_joint">
+  <joint type="fixed" name="base_to_laser_link_joint">
     <origin rpy="0 0 0" xyz="0.12 0 0.095"/>
-    <child link="laser"/>
+    <child link="laser_link"/>
     <parent link="base_link"/>
   </joint>
