Commit message: Nav tuning for scooba

File: scooba_base/urdf/scooba.xacro (robot description, xacro)
@@ -90,5 +90,5 @@
   </link>
   <joint type="fixed" name="base_to_laser_link_joint">
-    <origin rpy="0 0 0" xyz="0.1 0 0.1"/>
+    <origin rpy="0 0 0" xyz="0.1 -0.05 0.07"/>
     <child link="laser_link"/>
     <parent link="base_link"/>

Commit message: scooba urdf fixes

File: scooba_base/urdf/scooba.xacro (robot description, xacro)
@@ -4,5 +4,5 @@
   <xacro:property name="PI" value="3.1415926535897931"/>
   <!-- Import Rviz colors -->
-  <xacro:include filename="$(find scooba_base)/urdf/materials.xacro" />
+  <xacro:include filename="$(find office_bot)/urdf/materials.xacro" />
   <!-- Base Link -->
   <link name="base_link">
@@ -36,5 +36,5 @@
     </visual>
   </link>
-  <link name="left_wheel">
+  <link name="left_wheel_link">
     <collision name="collision">
       <origin xyz="0 0.0 0" rpy="0 1.5707 1.5707"/>
@@ -53,10 +53,10 @@
   <joint type="revolute" name="left_wheel_joint">
     <origin xyz="0 0.16 0.02" rpy="0 0 0"/>
-    <child link="left_wheel">left_wheel</child>
+    <child link="left_wheel_link">left_wheel</child>
     <parent link="base_link">base_link</parent>
     <axis xyz="0 1 0"/>
     <limit effort="100" velocity="100.0"  lower="-5000" upper="5000" />
   </joint>
-  <link name="right_wheel">
+  <link name="right_wheel_link">
     <collision name="collision">
       <origin xyz="0 0.0 0" rpy="0 1.5707 1.5707"/>
@@ -75,10 +75,10 @@
   <joint type="revolute" name="right_wheel_joint">
     <origin xyz="0 -0.16 0.02" rpy="0 0 0"/>
-    <child link="right_wheel">right_wheel</child>
+    <child link="right_wheel_link">right_wheel</child>
     <parent link="base_link">base_link</parent>
     <axis xyz="0 1 0"/>
     <limit effort="100" velocity="100.0"  lower="-5000" upper="5000" />
   </joint>
-  <link name="laser">
+  <link name="laser_link">
     <visual>
       <origin xyz="0 0.0 0" rpy="0 0 0"/>
@@ -89,22 +89,22 @@
     </visual>
   </link>
-  <joint type="fixed" name="laser_to_base_joint">
-    <origin rpy="0 0 0" xyz="-0.05 0 0.05"/>
-    <child link="laser"/>
+  <joint type="fixed" name="base_to_laser_link_joint">
+    <origin rpy="0 0 0" xyz="0.1 0 0.1"/>
+    <child link="laser_link"/>
     <parent link="base_link"/>
   </joint>
-  <link name="imu">
+  <link name="tango">
     <visual>
       <origin xyz="0 0.0 0" rpy="0 0 0"/>
       <geometry>
-        <cylinder length="0.01" radius="0.01"/>
+         <box size="0.2 0.12 0.01"/>
       </geometry>
       <material name="black"/>
     </visual>
   </link>
-  <joint type="fixed" name="imu_to_base_joint">
-    <origin rpy="0 0 -1.5708" xyz="0 0 0.06"/>
-    <child link="imu"/>
-    <parent link="base_link"/>
+  <joint type="fixed" name="tango_to_base_joint">
+    <origin rpy="0 1.571 1.571" xyz="0 -0.2 0.05"/>
+    <child link="base_link"/>
+    <parent link="tango"/>
   </joint>
 </robot>

Commit message: Assorted changes

File: scooba_base/urdf/scooba.xacro (robot description, xacro)
@@ -90,5 +90,5 @@
   </link>
   <joint type="fixed" name="base_to_laser_link_joint">
-    <origin rpy="0 0 0" xyz="0.1 -0.05 0.07"/>
+    <origin rpy="0 0 0" xyz="0.12 -0.05 0.09"/>
     <child link="laser_link"/>
     <parent link="base_link"/>
@@ -96,5 +96,5 @@
   <link name="tango">
     <visual>
-      <origin xyz="0 0.0 0" rpy="0 0 0"/>
+      <origin xyz="0 -0.05 0" rpy="0 0 0"/>
       <geometry>
          <box size="0.2 0.12 0.01"/>
@@ -108,3 +108,20 @@
     <parent link="tango"/>
   </joint>
+  <xacro:include filename="$(find office_bot)/urdf/optionally_adjustable_joint.urdf.xacro"/>
+  <link name="camera_link">
+    <visual>
+      <geometry>
+        <box size="0.03 0.04 0.04"/>
+      </geometry>
+      <material name="black"/>
+    </visual>
+    <visual>
+      <origin xyz="0 0 0.0" rpy="0 0 0"/>
+      <geometry>
+        <cylinder length="0.04" radius="0.01"/>
+      </geometry>
+      <material name="blue"/>
+    </visual>
+  </link>
+  <xacro:optionally_adjustable_joint link_name="camera_link" xyz="0.03 0.0 0.27" rpy="1.37 3.14 1.64" adjustable="false"/>
 </robot>

Commit message: Updated scooba urdf following changes to tango_nav_adaptor

File: scooba_base/urdf/scooba.xacro (robot description, xacro)
@@ -48,5 +48,5 @@
         <cylinder  length="0.015" radius="0.02"/>
       </geometry>
-      <material name="black"/>
+      <material name="grey"/>
     </visual>
   </link>
@@ -70,5 +70,5 @@
         <cylinder  length="0.015" radius="0.02"/>
       </geometry>
-      <material name="black"/>
+      <material name="grey"/>
     </visual>
   </link>
@@ -86,5 +86,5 @@
         <cylinder length="0.05" radius="0.03"/>
       </geometry>
-      <material name="black"/>
+      <material name="grey"/>
     </visual>
   </link>
@@ -96,13 +96,13 @@
   <link name="tango">
     <visual>
-      <origin xyz="0 -0.05 0" rpy="0 0 0"/>
+      <origin xyz="0 0 0.15" rpy="0 0 0"/>
       <geometry>
-         <box size="0.2 0.12 0.01"/>
+         <box size="0.01 0.2 0.12"/>
       </geometry>
-      <material name="black"/>
+      <material name="grey"/>
     </visual>
   </link>
   <joint type="fixed" name="tango_to_base_joint">
-    <origin rpy="0 1.571 1.571" xyz="0 -0.2 0.05"/>
+    <origin rpy="0 0 0" xyz="-0.05 0 0"/>
     <child link="base_link"/>
     <parent link="tango"/>
@@ -112,14 +112,14 @@
     <visual>
       <geometry>
-        <box size="0.03 0.04 0.04"/>
+        <box size="0.04 0.04 0.03"/>
       </geometry>
-      <material name="black"/>
+      <material name="grey"/>
     </visual>
     <visual>
-      <origin xyz="0 0 0.0" rpy="0 0 0"/>
+      <origin xyz="0 0 0.015" rpy="0 0 0"/>
       <geometry>
-        <cylinder length="0.04" radius="0.01"/>
+        <cylinder length="0.02" radius="0.01"/>
       </geometry>
-      <material name="blue"/>
+      <material name="grey"/>
     </visual>
   </link>
