Commit message: Added hokuyo to description

File: office_bot_description/urdf/office_bot.urdf.xacro (robot description, xacro)
@@ -2,8 +2,5 @@
 <robot name="roomba" xmlns:xacro="http://ros.org/wiki/xacro">
   <xacro:include filename="$(find ca_description)/urdf/create_2.urdf.xacro" />
-  <link name="laser_link"/>
-  <joint name="baser_to_laser_joint" type="fixed">
-    <parent link="base_link"/>
-    <child link="laser_link"/>
-  </joint>
+  <xacro:include filename="$(find office_bot_description)/urdf/hokuyo.urdf.xacro" />
+  <xacro:hokuyo_laser xyz="0 0 0.1" rpy="0 0 0" parent="base_link" />
 </robot>
